File: lisa-priam-datatower-card/lisa-priam-datatower-card.kicad_sch (KiCad schematic)
At the start: 8 parts

Commit message: updates - pcb created
Parts:
- added C1 (x14): 0.1uF 50V, Capacitor_THT_Custom:C_Disc_D7.0mm_W2.3mm_P5.00mm, symbol Device:C
- added J1: Lisa Expansion Card Edge, Connector_Custom:Apple_Lisa_ExpansionBus_CardEdge, symbol Connector_Custom:Apple_Lisa_ExpansionBus_CardEdge
- added P2: DB25_Receptacle_MountingHoles, Connector_Dsub:DSUB-25_Female_Horizontal_P2.77x2.84mm_EdgePinOffset4.94mm_Housed_MountingHolesOffset7.48mm, symbol Connector:DB25_Receptacle_MountingHoles
- added R2 (x8): 390, Resistor_THT_Custom:R_Axial_DIN0309_L9.0mm_D2.54mm_P12.70mm_Horizontal, symbol Device:R_US
- added R2 (x11): 330, Resistor_THT_Custom:R_Axial_DIN0309_L9.0mm_D2.54mm_P12.70mm_Horizontal, symbol Device:R_US
- added R2 (x4): 3.3K, Resistor_THT_Custom:R_Axial_DIN0309_L9.0mm_D2.54mm_P12.70mm_Horizontal, symbol Device:R_US
- added R2 (x3): 220, Resistor_THT_Custom:R_Axial_DIN0309_L9.0mm_D2.54mm_P12.70mm_Horizontal, symbol Device:R_US
- added UA4: 74LS164, Package_DIP:DIP-14_W7.62mm, symbol 74xx_Custom:74LS164
- added UA5: 74LS02, Package_DIP:DIP-14_W7.62mm, symbol 74xx:74LS02
- added UB2: 74LS112, Package_DIP:DIP-16_W7.62mm, symbol 74xx:74LS112
- added UC1: 74LS125, Package_DIP:DIP-14_W7.62mm, symbol 74xx:74LS125
- added UC3: 74LS132, Package_DIP:DIP-14_W7.62mm, symbol 74xx:74LS132
- added UC4, UD1: 74LS00, Package_DIP:DIP-14_W7.62mm, symbol 74xx:74LS00
- added UC6: 75463, Package_DIP:DIP-8_W7.62mm, symbol 75xx_Custom:75463
- added UD2: 2716, Package_DIP:DIP-24_W15.24mm, symbol Memory_EPROM_Custom:2716
- added UD4: 8304, Package_DIP:DIP-20_W7.62mm, symbol 8xxx_Custom:8304
- added UE1, UE4, UE5, UE6, UE7: 74LS374, Package_DIP:DIP-20_W7.62mm, symbol 74xx:74LS374
- added UE2: 74LS280, Package_DIP:DIP-14_W7.62mm, symbol 74xx:74LS280
- added UE3: 74LS244, Package_DIP:DIP-20_W7.62mm, symbol 74xx:74LS244
- UB1, UC2: footprint (none) -> Package_DIP:DIP-14_W7.62mm
- UB3, UB4, UB7: footprint (none) -> Package_DIP:DIP-16_W7.62mm
Connections:
- net BA9: now also J1.39 (BA9), UD2.23 (A8)
- net CPUCK: now also J1.8 (CPUCK)
- net GND: now also UB1.7 (GND), UB3.8 (GND), UB4.2 (K), UB4.8 (GND), UB5.4 (GND), UB6.4 (GND), UB7.8 (GND), UC2.7 (GND), UC5.4 (GND), C1.1, C1.1, C1.1, C1.1, C1.1, C1.1, C1.1, C1.1, C1.1, C1.1, C1.1, C1.1, C1.1, C1.1, J1.53 (GND), J1.54 (GND), P2.0 (PAD), P2.1, P2.2, P2.20 (P20), P2.24 (P24), P2.4, P2.9, R2.1, R2.1, R2.1, R2.1, R2.1, R2.1, R2.1, R2.1, R2.2, R2.2, R2.2, UA4.7 (GND), UA5.7 (GND), UB2.8 (GND), UC1.5, UC1.7 (GND), UC3.7 (GND), UC4.7 (GND), UC6.4 (GND), UD1.7 (GND), UD2.12 (GND), UD2.18 (/CE), UD2.20 (/OE), UD4.10 (GND), UE1.1 (OE), UE1.10 (GND), UE2.7 (GND), UE3.10 (GND), UE4.10 (GND), UE5.10 (GND), UE6.10 (GND), UE7.10 (GND)
- net HAD0: now also P2.16 (P16)
- net HAD1: now also P2.17 (P17)
- net HAD2: now also P2.19 (P19)
- net HUNK: now also P2.14 (P14)
- net LA1: now also UE1.2 (O0)
- net LA2: now also UE1.5 (O1)
- net LA3: now also UE1.6 (O2)
- net LA4: now also UE1.9 (O3)
- net PU1: now also R2.2
- net PU5: now also R2.2, UB2.10 (~{S}), UB2.12 (K), UB2.2 (K), UB2.4 (~{S})
- net /BUSE: now also UD4.9 (CD)
- net /FFR: now also UA4.9 (/CLR), UB2.14 (~{R}), UB2.15 (~{R}), UD1.1
- net /HRST: now also P2.21 (P21)
- net /RESET: now also J1.7 (/RESET)
- net /SH: now also UB1.11, UB1.12, UC2.1, UC2.9, UC1.10
- net +5V: now reaches UB1.14 (VCC)
- net +5V: now also UB3.16 (VCC), UB4.16 (VCC), UB5.8 (VCC), UB6.8 (VCC), UB7.16 (VCC), UC2.14 (VCC), UC5.8 (VCC), C1.2, C1.2, C1.2, C1.2, C1.2, C1.2, C1.2, C1.2, C1.2, C1.2, C1.2, C1.2, C1.2, C1.2, J1.55 (+5V), J1.56 (+5V), R2.1, R2.1, R2.1, R2.1, R2.1, R2.2, R2.2, R2.2, R2.2, R2.2, R2.2, R2.2, R2.2, R2.2, R2.2, UA4.14 (VCC), UA5.14 (VCC), UB2.16 (VCC), UC1.14 (VCC), UC3.14 (VCC), UC4.14 (VCC), UC6.8 (VCC), UD1.14 (VCC), UD2.21 (VPP), UD2.24 (VCC), UD4.20 (VCC), UE1.20 (VCC), UE2.14 (VCC), UE3.20 (VCC), UE4.20 (VCC), UE5.20 (VCC), UE6.20 (VCC), UE7.20 (VCC)
- net /SL: now reaches UC2.4
- net /SL: now also UC1.4
- net at UC2.5: now also UC2.10, UC3.6
- net /LORD: now reaches UC2.6
- net /LORD: now also UC1.1, UE3.1 (OEa), UE3.19 (OEb)
- net at UB1.8, UB7.6 (~{Q}): now also UB3.1 (C)
- net at UB4.12 (K): now also UB1.2, UB2.9 (Q), UC4.13, UC4.5, UD1.12
- net at UB4.13 (C), UB7.9 (Q): now also UA4.8 (CLK), UB2.1 (C), UB2.13 (C)
- net READ: now reaches UC2.2
- net READ: now also J1.48 (READ), UC3.4, UC3.5
- net /HIWR: now reaches UC2.3
- net /HIWR: now also UD1.5
- net /HIRD: now reaches UC2.8
- net /HIRD: now also UE5.1 (OE), UE7.1 (OE)
- net at UB1.1: now also UC1.9
- net at UB1.3: now also UB1.4
- net SHI: now reaches UB1.13
- net SHI: now also UE1.11 (Cp), UE4.11 (Cp), UE6.11 (Cp)
- net at UC5.1: now also UC3.2, UC6.6, UD1.3, UD1.4
- net POUT: now reaches UC5.2
- net POUT: now also UB4.3 (J), UE2.5 (Even)
- net HCBUSP: now reaches UC5.3
- net HCBUSP: now also P2.18 (P18), R2.1, R2.2, UC3.1
- net BA6: now reaches UB1.5
- net BA6: now also UB1.6, J1.36 (BA6), UD2.3 (A5), UE1.14 (D5)
- net at UB3.15 (~{R}): now also UD1.11
- net at UB3.2 (K): now also UB3.3 (J), UD1.8
- net PU2: now reaches UB3.4 (~{S})
- net PU2: now also R2.2
- net CKP: now reaches UB3.5 (Q)
- net CKP: now also UB4.1 (C), UC4.10, UC4.12
- net at UB3.6 (~{Q}): now also UC6.1, UC6.7
- net LA5: now reaches UB4.15 (~{R})
- net LA5: now also UE1.12 (O4)
- net at UB4.4 (~{S}): now also R2.1
- net at UB4.5 (Q): now also UC1.2
- new net: UC3.10, UC3.11
- new net: J1.13 (/BGINn), J1.14 (/BGOUTn)
- new net: J1.44 (/VPA), J1.6 (/IAKn)
- new net: UA5.1, UB2.3 (J)
- new net: UA4.1 (A), UA4.2 (B), UB2.5 (Q), UC4.1, UC4.9
- new net: UB2.6 (~{Q}), UD1.10
- new net: UD2.14 (D4), UE3.11 (I0b)
- new net: UD2.15 (D5), UE3.13 (I1b)
- new net: UD2.16 (D6), UE3.15 (I2b)
- new net: UD2.17 (D7), UE3.17 (I3b)
- new net: UD2.9 (D0), UE3.2 (I0a)
- new net: UD2.10 (D1), UE3.4 (I1a)
- new net: UD2.11 (D2), UE3.6 (I2a)
- new net: UD2.13 (D3), UE3.8 (I3a)
- new net: UA4.4 (Qb), UA5.2, UB2.11 (J)
- new net: UA4.5 (Qc), UA5.3
- new net: UB2.7 (~{Q}), UD1.9
- new net BA1: J1.31 (BA1), UD2.8 (A0), UE1.3 (D0)
- new net BA2: J1.32 (BA2), UD2.7 (A1), UE1.4 (D1)
- new net BA3: J1.33 (BA3), UD2.6 (A2), UE1.7 (D2)
- new net BA4: J1.34 (BA4), UD2.5 (A3), UE1.8 (D3)
- new net BA5: J1.35 (BA5), UD2.4 (A4), UE1.13 (D4)
- new net BA7: J1.37 (BA7), UD2.2 (A6), UE1.17 (D6)
- new net BA8: J1.38 (BA8), UD2.1 (A7), UE1.18 (D7)
- new net BAA: J1.40 (BA10), UD2.22 (A9)
- new net BAB: J1.41 (BA11), UD2.19 (A10)
- new net BD0: J1.30 (BD0), UE3.18 (O0a), UE4.3 (D0), UE5.2 (O0)
- new net BD1: J1.29 (BD1), UE3.16 (O1a), UE4.4 (D1), UE5.5 (O1)
- new net BD2: J1.28 (BD2), UE3.14 (O2a), UE4.7 (D2), UE5.6 (O2)
- new net BD3: J1.27 (BD3), UE3.12 (O3a), UE4.8 (D3), UE5.9 (O3)
- new net BD4: J1.26 (BD4), UE3.9 (O0b), UE4.13 (D4), UE5.12 (O4)
- new net BD5: J1.25 (BD5), UE3.7 (O1b), UE4.14 (D5), UE5.15 (O5)
- new net BD6: J1.24 (BD6), UE3.5 (O2b), UE4.17 (D6), UE5.16 (O6)
- new net BD7: J1.23 (BD7), UE3.3 (O3b), UE4.18 (D7), UE5.19 (O7)
- new net BD8: J1.22 (BD8), UE6.3 (D0), UE7.2 (O0)
- new net BD9: J1.21 (BD9), UE6.4 (D1), UE7.5 (O1)
- new net BDA: J1.20 (BD10), UE6.7 (D2), UE7.6 (O2)
- new net BDB: J1.19 (BD11), UE6.8 (D3), UE7.9 (O3)
- new net BDC: J1.18 (BD12), UE6.13 (D4), UE7.12 (O4)
- new net BDD: J1.17 (BD13), UE6.14 (D5), UE7.15 (O5)
- new net BDE: J1.16 (BD14), UE6.17 (D6), UE7.16 (O6)
- new net BDF: J1.15 (BD15), UC1.3, UE6.18 (D7), UE7.19 (O7)
- new net CKH: UC4.8, UE7.11 (Cp)
- new net CKL: UC4.11, UE5.11 (Cp)
- new net HCBUS0: P2.5, R2.1, R2.2, UD4.19 (B0)
- new net HCBUS1: P2.6, R2.1, R2.2, UD4.18 (B1)
- new net HCBUS2: P2.8, R2.1, R2.2, UD4.17 (B2)
- new net HCBUS3: P2.22 (P22), R2.1, R2.2, UD4.16 (B3)
- new net HCBUS4: P2.23 (P23), R2.1, R2.2, UD4.15 (B4)
- new net HCBUS5: P2.11, R2.1, R2.2, UD4.14 (B5)
- new net HCBUS6: P2.12, R2.1, R2.2, UD4.13 (B6)
- new net HCBUS7: P2.13, R2.1, R2.2, UD4.12 (B7)
- new net LA6: UE1.15 (O5)
- new net LA7: UD1.13, UE1.16 (O6)
- new net LA8: UC3.9, UE1.19 (O7)
- new net LD0: UD4.1 (A0), UE2.8 (A), UE4.2 (O0), UE5.3 (D0), UE6.2 (O0), UE7.3 (D0)
- new net LD1: UD4.2 (A1), UE2.9 (B), UE4.5 (O1), UE5.4 (D1), UE6.5 (O1), UE7.4 (D1)
- new net LD2: UD4.3 (A2), UE2.10 (C), UE4.6 (O2), UE5.7 (D2), UE6.6 (O2), UE7.7 (D2)
- new net LD3: UD4.4 (A3), UE2.11 (D), UE4.9 (O3), UE5.8 (D3), UE6.9 (O3), UE7.8 (D3)
- new net LD4: UD4.5 (A4), UE2.12 (E), UE4.12 (O4), UE5.13 (D4), UE6.12 (O4), UE7.13 (D4)
- new net LD5: UD4.6 (A5), UE2.13 (F), UE4.15 (O5), UE5.14 (D5), UE6.15 (O5), UE7.14 (D5)
- new net LD6: UD4.7 (A6), UE2.1 (G), UE4.16 (O6), UE5.17 (D6), UE6.16 (O6), UE7.17 (D6)
- new net LD7: UD4.8 (A7), UE2.2 (H), UE4.19 (O7), UE5.18 (D7), UE6.19 (O7), UE7.18 (D7)
- new net PIN: UC3.3, UE2.4 (I)
- new net WR: UC4.2, UC4.4, UC6.2, UD1.2, UD1.6, UD4.11 (T/R)
- new net /BTREQ: P2.10, R2.1, R2.2, UC3.12
- new net /DTACK: J1.46 (/DTACK), UC1.6, UC1.8
- new net /HIR: P2.25 (P25), R2.1, R2.1, UC3.13
- new net /HRD: P2.15 (P15), UC6.3
- new net /HWR: P2.3, UC6.5
- new net /INTn: J1.5 (/INTn), UC3.8
- new net /OEH: UC4.3, UE6.1 (OE)
- new net /OEL: UC4.6, UE4.1 (OE)
- new net /SHn: J1.4 (/SHn)
- new net /SLn: J1.3 (/SLn)
- no-connect marks 2 -> 37
Other:
- note added: "DECOUPLING CAPACITORS"
- note added: "POWER CONNECTIONS"
- note added: "UNUSED"
- moved on the sheet: UB1A, UB1B, UB1C, UB1D, UB1E, UB3A, UB3B, UB3C, UB4A, UB4B, UB4C, UB5A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
